File: STM_proto_board_active_filters.kicad_pcb (KiCad board)
At the start: 2 copper layers, 40.7 x 81.1 mm, 95 parts, among them J1 Conn_02x07, J2 Conn_02x07, J3 Conn_02x07, U1 TL072, U2 TL072, U3 TL072

Commit message: Add information on PCB and schematic
Other:
- board text added: "Patryk 22.12.2025 rev: 0.0.1"
- board text removed: "PW"
