File: STM_proto_board_active_filters.kicad_sch (KiCad schematic)
At the start: 95 parts, among them J1 Conn_02x07, J2 Conn_02x07, J3 Conn_02x07, U1 TL072, U2 TL072, U3 TL072

Commit message: Add information on PCB and schematic
Other:
- company: (none) -> KN NaMi
- title: (none) -> main schematic
Changed lines of the file:
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@@
 	(generator_version "9.0")
 	(paper "A3")
+	(title_block
+		(title "main schematic")
+		(date "2025-12-22")
+		(rev "0.0.1")
+		(company "KN NaMi")
+	)
 	(text "https://www.electronics-tutorials.ws/opamp/opamp_2.html"
 		(exclude_from_sim no)
