File: NaMi DevBoard active filters/NaMi DevBoard active filters.kicad_pcb (KiCad board)
At the start: 2 copper layers, 40.7 x 81.1 mm, 95 parts, among them J1 Conn_02x07, J2 Conn_02x07, J3 Conn_02x07, U1 TL072, U2 TL072, U3 TL072

Commit message: date change
Other:
- board text added: "Patryk 15.01.2026 rev: 0.0.2"
- board text removed: "Patryk 13.01.2026 rev: 0.0.2"
Changed lines of the file:
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@@
 		(layer "Edge.Cuts")
 	)
-	(gr_text "Patryk\n13.01.2026\nrev: 0.0.2"
+	(gr_text "Patryk\n15.01.2026\nrev: 0.0.2"
 		(at 70.6 119.5 90)
 		(layer "B.Cu" knockout)
